Commit message: Can navigate inefficient to a point

File: agv_pkg/urdf/base.xacro (robot description, xacro)
@@ -210,9 +210,5 @@
         <origin rpy="0 0 0" xyz="0.0 0.0 0.0"/>
     </xacro:sensor_imu>
-    <!-- LIDAR -->
-    <xacro:sensor_lidar
-        name="rplidar_front"
-        parent_link="chassis_link"
-        chassis_top_relative_height="${0.5 * chassis_height}" />
+    <xacro:include filename="lidar.xacro" />
     <!-- Bump -->
     <!-- Sonar -->

File: agv_pkg/urdf/gazebo.xacro (robot description, xacro)
@@ -97,5 +97,5 @@
                     <scan>
                         <horizontal>
-                            <samples>640</samples>
+                            <samples>360</samples>
                             <resolution>1.0</resolution>
                             <min_angle>${-pi}</min_angle>
@@ -115,4 +115,9 @@
                     </range>
                 </lidar>
+                <!-- <plugin
+                    filename="libignition-gazebo-sensors-system.so"
+                    name="ignition::gazebo::systems::Sensors">
+                    <render_engine>ogre2</render_engine>
+                </plugin> -->
             </sensor>
         </gazebo>
@@ -131,20 +136,14 @@
     <xacro:gazebo_sensor_rplidar name="rplidar_front" />
     <gazebo>
-        <plugin
-                filename="gz-sim-joint-state-publisher-system"
-                name="gz::sim::systems::JointStatePublisher">
-            <parameters>$(find agv_pkg)/config/zinger.yaml</parameters>
+        <plugin name="gz_ros2_control::GazeboSimROS2ControlPlugin" filename="libgz_ros2_control-system.so">
+            <parameters>$(find agv_pkg)/config/my_controllers.yaml</parameters>
+            <parameters>$(find agv_pkg)/config/gaz_ros2_ctl_use_sim.yaml</parameters>
         </plugin>
     </gazebo>
     <gazebo>
-        <plugin name="gz_ros2_control::GazeboSimROS2ControlPlugin" filename="libgz_ros2_control-system.so">
-            <parameters>$(find agv_pkg)/config/zinger.yaml</parameters>
-            <parameters>$(find agv_pkg)/config/gaz_ros2_ctl_use_sim.yaml</parameters>
-        </plugin>
-    </gazebo>
-         <!-- <plugin
-                filename="libignition-gazebo-pose-publisher-system.so"
-                name="gz::sim::systems::JointStatePublisher">
-            <publish_link_pose>true</publish_link_pose>
+         <plugin filename="gz-sim-joint-state-publisher-system"
+            name="gz::sim::systems::JointStatePublisher">
+            <parameters>$(find agv_pkg)/config/my_controllers.yaml</parameters>
+            <!-- <publish_link_pose>true</publish_link_pose>
             <publish_sensor_pose>true</publish_sensor_pose>
             <publish_collision_pose>false</publish_collision_pose>
@@ -154,5 +153,6 @@
             <use_pose_vector_msg>true</use_pose_vector_msg>
             <static_publisher>true</static_publisher>
-            <static_update_frequency>-1</static_update_frequency>
-        </plugin> -->
+            <static_update_frequency>-1</static_update_frequency> -->
+        </plugin>
+    </gazebo>
 </robot>

File: agv_pkg/urdf/macros.xacro (robot description, xacro)
@@ -203,5 +203,5 @@
     </xacro:macro>
     <!-- Lidar sensor -->
-    <xacro:macro name="sensor_lidar" params="name parent_link chassis_top_relative_height">
+    <!-- <xacro:macro name="sensor_lidar" params="name parent_link chassis_top_relative_height">
         <xacro:property name="mass"     value="0.17"/>
         <xacro:property name="length_x" value="0.071" />
@@ -241,5 +241,5 @@
             </inertial>
         </link>
-    </xacro:macro>
+    </xacro:macro> -->
     <!-- Bump sensor -->
     <!-- Sonar sensor -->
