Commit message: Real lidar added

File: src/agv_pkg/description/lidar.xacro (robot description, xacro)
@@ -1,61 +1,11 @@
 <?xml version="1.0"?>
-<robot xmlns:xacro="http://www.ros.org/wiki/xacro" >
-    <xacro:macro name="inertial_cylinder" params="mass length radius *origin">
-        <inertial>
-            <xacro:insert_block name="origin"/>
-            <mass value="${mass}" />
-            <inertia ixx="${(1/12) * mass * (3*radius*radius + length*length)}" ixy="0.0" ixz="0.0"
-                    iyy="${(1/12) * mass * (3*radius*radius + length*length)}" iyz="0.0"
-                    izz="${(1/2) * mass * (radius*radius)}" />
-        </inertial>
-    </xacro:macro>
-    <joint name="laser_joint" type="fixed">
-        <parent link="chassis_link"/>
-        <child link="laser_frame"/>
-        <origin xyz="0.28 0 -0.1" rpy="0 0 0"/>
+<robot xmlns:xacro="http://www.ros.org/wiki/xacro" name="robot">
+  <xacro:include filename="$(find ldlidar_node)/urdf/ldlidar_descr.urdf.xml" />
+  <xacro:macro name="add_lidar_mount" params="parent_link">
+    <joint name="ldlidar_mount_joint" type="fixed">
+      <parent link="${parent_link}"/>
+      <child link="ldlidar_base"/>
+      <origin xyz="0.28 0 -0.11" rpy="0 0 -1.5708"/>
     </joint>
-    <link name="laser_frame">
-        <visual>
-            <geometry>
-                <cylinder radius="0.02" length="0.03"/>
-            </geometry>
-        </visual>
-        <visual>
-            <origin xyz="0 0 -0.05"/>
-            <geometry>
-                <cylinder radius="0.01" length="0.1"/>
-            </geometry>
-        </visual>
-        <collision>
-            <geometry>
-                <cylinder radius="0.05" length="0.04"/>
-            </geometry>
-        </collision>
-        <xacro:inertial_cylinder mass="0.1" length="0.04" radius="0.03">
-            <origin xyz="0 0 0" rpy="0 0 0"/>
-        </xacro:inertial_cylinder>
-    </link>
-    <gazebo reference="laser_frame">
-        <material>Gazebo/Black</material>
-        <sensor name="laser" type="gpu_lidar">
-            <pose> 0 0 0 0 0 0 </pose>
-            <visualize>false</visualize>
-            <update_rate>10</update_rate>
-            <lidar>
-                <scan>
-                    <horizontal>
-                        <samples>360</samples>
-                        <min_angle>-3.14</min_angle>
-                        <max_angle>3.14</max_angle>
-                    </horizontal>
-                </scan>
-                <range>
-                    <min>0.3</min>
-                    <max>12</max>
-                </range>
-            </lidar>
-            <topic>scan</topic>
-            <gz_frame_id>laser_frame</gz_frame_id>
-        </sensor>
-    </gazebo>
+  </xacro:macro>
 </robot>

File: src/agv_pkg/description/robot.urdf.xacro (robot description, xacro)
@@ -2,13 +2,20 @@
 <robot xmlns:xacro="http://www.ros.org/wiki/xacro"  name="robot">
     <xacro:arg name="use_ros2_control" default="true"/>
-    <xacro:arg name="is_simulation" default="false"/>
+    <xacro:arg name="is_simulation" default="true"/>
     <xacro:include filename="robot.urdf"/>
+    <xacro:if value="$(arg is_simulation)">
+        <xacro:include filename="lidar_gazebo.xacro" />
+    </xacro:if>
+    <xacro:unless value="$(arg is_simulation)">
+        <xacro:include filename="lidar.xacro" />
+        <xacro:add_lidar_mount parent_link="chassis_link"/>
+    </xacro:unless>
      <xacro:if value="$(arg use_ros2_control)">
         <xacro:include filename="ros2_control.xacro" />
+        <!-- <xacro:include filename="gazebo_control.xacro" /> -->
     </xacro:if>
     <xacro:unless value="$(arg use_ros2_control)">
         <xacro:include filename="gazebo_control.xacro" />
     </xacro:unless>
-    <xacro:include filename="lidar.xacro" />
-    <xacro:include filename="cameras.xacro" />
+    <!-- <xacro:include filename="cameras.xacro" /> -->
 </robot>

File: src/agv_pkg/urdf/base.xacro (robot description, xacro)
@@ -94,5 +94,5 @@
             <mass value="${chassis_mass}"/>
             <inertia
-                ixx="${chassis_mass / 12.0 * (chassis_width * chassis_width + chassis_height * chassis_height)}"
+                ixx="${(chassis_mass / 12.0 * (chassis_width * chassis_width + chassis_height * chassis_height))}"
                 ixy="0"
                 ixz="0"
